File: bldc-hardware-master/design/BLDC_4.kicad_pcb (KiCad board)
At the start: 4 copper layers, 100 x 54.3 mm, 129 parts, among them J1 RJ45-8N-B, J2 Conn_01x02_Male, J3 Conn_01x02_Male, K1 SERVO, P1 HALL/Encoder, P101 CANBUS, P2 SWD, P3 PWR_COMM, P4 IN+, P5 IN-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

Commit message: Update BLDC_4.kicad_pcb
Parts:
- removed REF** (x3): MountingHole_4mm, MountingHole:MountingHole_4mm
- added  : MountingHole_4mm, MountingHole:MountingHole_4mm, F.Cu at (111.8, 88.9)
- added  : MountingHole_4mm, MountingHole:MountingHole_4mm, F.Cu at (111.8, 44.5)
- added  : MountingHole_4mm, MountingHole:MountingHole_4mm, F.Cu at (21.6, 44.5)
Other:
- board text added: "SEM 2020 Girton Grammar School"
Changed lines of the file:
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@@
   (general
     (thickness 1.6)
-    (drawings 45)
+    (drawings 46)
     (tracks 1918)
     (zones 0)
@@
   )
   (setup
-    (last_trace_width 0.889)
+    (last_trace_width 0.2032)
     (user_trace_width 0.254)
     (user_trace_width 0.3048)
@@
     (tags "mounting hole 4mm no annular")
     (attr virtual)
-    (fp_text reference REF** (at 0 -5) (layer F.SilkS)
+    (fp_text reference " " (at 0 -5) (layer F.SilkS)
       (effects (font (size 1 1) (thickness 0.15)))
     )
@@
     (tags "mounting hole 4mm no annular")
     (attr virtual)
-    (fp_text reference REF** (at 0 -5) (layer F.SilkS)
+    (fp_text reference " " (at 0 -5) (layer F.SilkS)
       (effects (font (size 1 1) (thickness 0.15)))
     )
@@
     (tags "mounting hole 4mm no annular")
     (attr virtual)
-    (fp_text reference REF** (at 0 -5) (layer F.SilkS)
+    (fp_text reference " " (at 0 -5) (layer F.SilkS)
       (effects (font (size 1 1) (thickness 0.15)))
     )
@@
     )
   )
+  (gr_text "SEM 2020\nGirton Grammar School " (at 93.98 88.9) (layer F.SilkS)
+    (effects (font (size 1 1) (thickness 0.25)))
+  )
   (gr_text +12V (at 20.32 64.77 90) (layer F.SilkS)
